File: hardware/kicad/ssr4/circuit.kicad_pcb (KiCad board)
At the start: 2 copper layers, 90 x 75 mm, 81 parts, among them J1 USB_C_Receptacle_USB2.0_16P, K1 CPC40055ST, K2 CPC40055ST, K3 CPC40055ST, K4 CPC40055ST, Q1 AO3400A, Q2 AO3400A, Q3 AO3400A, Q4 AO3400A, Q5 AO3400A, SW1 SW_Push, SW2 SW_Push, U1 ESP32-C3-MINI-1-H4X, U2 AMS1117-3.3, U3 USBLC6-2SC6, U7 TMP302ADRLR, X1 Screw_Terminal_01x02, X2 Screw_Terminal_01x02, X3 Screw_Terminal_01x02, X4 Screw_Terminal_01x02, X5 Screw_Terminal_01x02

Commit message: fix(hardware): remove a ground via touching the antenna keep-out
A GND stitching via overlapped the ESP32-C3 antenna keep-out by 0.02 mm;
KiCad 10.0.7's DRC in CI flagged it. Regenerated board, fabrication
packages and validation reports without it.
Routing:
- net GND: vias 90 -> 89
Changed lines of the file:
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@@
-	)
-	(via
-		(at 113.15 123.15)
-		(size 0.6)
-		(drill 0.3)
-		(layers "F.Cu" "B.Cu")
-		(net "GND")
 	)
 	(via
